Commit message: not working but wanna delet everhing

File: niagara_model/urdf/Robot_2.urdf (robot description, URDF)
Before this commit: robot niagara_car, 9 links, 8 joints
Links:
- link base_link: mass 396.320233140643 -> 1.0
- link left_front: mass 87.7464239263491 -> 1.0
- link left_rear: mass 87.7464239263501 -> 1.0
- link right_front: mass 87.7464239239315 -> 1.0
- link right_rear: mass 87.7464239263518 -> 1.0
