Commit message: error of the robot resolved.

File: niagara_model/urdf/VLP-16.xacro (robot description, xacro)
@@ -17,4 +17,5 @@
         <geometry>
           <cylinder length="0.073" radius="0.04" />
+          <!-- <mesh filename="file://$(find niagara_model)/meshes/os1_64.dae" /> -->
         </geometry>
       </visual>
@@ -28,4 +29,5 @@
         <geometry>
           <cylinder radius="0.0516" length="0.0717"/>
+          <!-- <mesh filename="file://$(find niagara_model)/meshes/os1_64.dae" /> -->
         </geometry>
       </collision>
@@ -45,5 +47,5 @@
         <origin xyz="0 0 -0.0377"/>
         <geometry>
-          <!-- <mesh filename="$(find niagara_model)/meshes/os1_64.dae"/> -->
+          <!-- <mesh filename="file://$(find niagara_model)/meshes/os1_64.dae" /> -->
           <cylinder length="0.073" radius="0.04" />
         </geometry>
