Commit message: susoetion added

File: niagara_model/urdf/Autoreifen.xacro (robot description, xacro)
@@ -1,3 +1,240 @@
 <?xml version="1.0"?>
 <robot name="dasautonomeauto" xmlns:xacro="http://www.ros.org/wiki/xacro">
+  <!-- hub_dia and tire_dia are the diameters of the hub and tire,
+       respectively. hex_hub_depth is the distance that the hex hub is
+       inset from the outer edge of the tire. It is set so that each wheel
+       is a "zero offset" wheel. hex_hub_depth = tire_width / 2 -
+       axle_length. -->
+    <xacro:property name="tire_dia" value="0.350"/>  <!-- Reduced from 0.440 -->
+    <xacro:property name="tire_width" value="0.195"/>  <!-- Reduced from 0.195 -->
+    <xacro:property name="hub_dia" value="0.235"/>  <!-- Reduced from 0.235 -->
+  <xacro:property name="hex_hub_depth" value="0.120"/> <!-- or +0.072 -->
+  <xacro:property name="wheel_mass" value="8.0"/>   <!-- check -->
+  <!-- hex_hub_dist is the distance between left and right hex hubs when
+       the shock absorbers are fully extended. axle_length is the distance
+       from a U joint to the corresponding hex hub. wheel_travel is the
+       vertical wheel travel. -->
+  <xacro:property name="wheelbase" value="2.1"/>
+  <xacro:property name="hex_hub_dist" value="0.9191"/>  <!-- 1.127 0.742 0.900 check -->
+  <xacro:property name="axle_length" value="0.120"/>
+  <xacro:property name="wheel_travel" value="0.209492959255614"/>
+  <xacro:property name="shock_z_offset" value="0.10"/>
+  <!-- Degree-to-radian conversions -->
+  <xacro:property name="degrees_45" value="0.785398163"/>
+  <xacro:property name="degrees_90" value="1.57079633"/>
+  <xacro:property name="degrees_180" value="3.14159265"/>
+  <!-- shock_eff_limit is 2 * ((shock_stroke / 2) * shock_spring_constant) N. -->
+  <xacro:property name="shock_eff_limit" value="100"/>
+  <xacro:property name="shock_vel_limit" value="1000"/>
+  <xacro:property name="wheel_joint_damping" value="0.2" />
+  <xacro:property name="wheel_joint_friction" value="0.7" />
+  <xacro:property name="suspension_joint_damping" value="0.2" />
+  <xacro:property name="suspension_joint_friction" value="0.7" />
+  <!-- axle eff limit = 2 * stall_torque
+       as a function of the max gradient (15%) with overall max payload (600Kg) * wheel_radius
+       (calculating this way, it should be divided by 2 if 2 motors are used)
+       axle_eff_limit = 204.95 / 2 N m = ~102.5 -->
+  <!-- xacro:property name="axle_eff_limit" value="102.5"/ -->
+  <xacro:property name="axle_eff_limit" value="204.95"/>
+  <!-- max_speed = 33 Km/h = 9.17 m/s
+       axle_vel_limit = (2 * pi) * (max_speed / (pi * tire_dia)) =  39.02 rad/s -->
+  <xacro:property name="axle_vel_limit" value="39.02"/>
+  <!-- Servo_stall_torque of the direction axis in Nm. servo_no_load_speed is
+       measured in rad/s. -->
+  <xacro:property name="servo_stall_torque" value="50"/>  <!-- check -->
+  <xacro:property name="servo_no_load_speed" value="25"/> <!-- check -->
+  <!-- Inertia of a thick-walled cylindrical tube with open ends. Height is
+       measured along the z axis, which is the tube's axis. inner_rad and
+       outer_rad are the tube's inner and outer radii, respectively. -->
+  <xacro:macro name="thick_walled_tube_inertial"
+               params="inner_rad outer_rad height mass">
+    <inertial>
+      <mass value="${mass}"/>
+      <inertia ixx="${(1 / 12) * mass * (3 * (inner_rad * inner_rad +
+                    outer_rad * outer_rad) + height * height)}"
+               ixy="0" ixz="0"
+               iyy="${(1 / 12) * mass * (3 * (inner_rad * inner_rad +
+                    outer_rad * outer_rad) + height * height)}"
+               iyz="0"
+               izz="${mass * (inner_rad * inner_rad +
+                    outer_rad * outer_rad) / 2}"/>
+    </inertial>
+  </xacro:macro>
+  <!-- Null inertial element. This is needed to make the model work with
+       Gazebo. -->
+  <xacro:macro name="null_inertial">
+    <inertial>
+      <mass value="0.001"/>
+      <inertia ixx="0.001" ixy="0" ixz="0" iyy="0.001" iyz="0" izz="0.001"/>
+    </inertial>
+  </xacro:macro>
+  <!-- Shock absorber -->
+  <xacro:macro name="shock"
+               params="lr_prefix fr_prefix lr_reflect fr_reflect child">
+    <joint name="${lr_prefix}_${fr_prefix}_shock" type="prismatic">
+      <parent link="base_link"/>
+      <child link="${child}"/>
+      <origin xyz="${fr_reflect * wheelbase / 2}
+                   ${lr_reflect * ((hex_hub_dist / 2) - axle_length)}
+                   ${-wheel_travel}"/>
+                  <!-- ${(wheel_travel / 2) - shock_z_offset}"/-->
+      <axis xyz="0 0 -1"/>
+      <limit lower="${-wheel_travel / 2}" upper="${wheel_travel / 2}"
+             effort="${shock_eff_limit}" velocity="${shock_vel_limit}"/>
+      <joint_properties damping="${suspension_joint_damping}" friction="{suspension_joint_friction}"/>
+    </joint>
+    <transmission name="${lr_prefix}_${fr_prefix}_shock_trans">
+      <type>transmission_interface/SimpleTransmission</type>
+      <joint name="${lr_prefix}_${fr_prefix}_shock">
+        <hardwareInterface>hardware_interface/EffortJointInterface</hardwareInterface>
+      </joint>
+      <actuator name="${lr_prefix}_${fr_prefix}_shock_act">
+        <mechanicalReduction>1</mechanicalReduction>
+      </actuator>
+    </transmission>
+  </xacro:macro>
+  <!-- Shock absorber for the front wheels -->
+  <xacro:macro name="shock_front"
+               params="lr_prefix fr_prefix lr_reflect fr_reflect child">
+    <joint name="${lr_prefix}_${fr_prefix}_shock" type="prismatic">
+      <parent link="base_link"/>
+      <child link="${child}"/>
+      <origin xyz="${fr_reflect * 0.90902595238888}
+                   ${lr_reflect * ((hex_hub_dist / 2) - axle_length)}
+                   ${-wheel_travel}"/>
+                  <!-- ${(wheel_travel / 2) - shock_z_offset}"/-->
+      <axis xyz="0 0 -1"/>
+      <limit lower="${-wheel_travel / 2}" upper="${wheel_travel / 2}"
+             effort="${shock_eff_limit}" velocity="${shock_vel_limit}"/>
+      <joint_properties damping="${suspension_joint_damping}" friction="{suspension_joint_friction}"/>
+    </joint>
+    <transmission name="${lr_prefix}_${fr_prefix}_shock_trans">
+      <type>transmission_interface/SimpleTransmission</type>
+      <joint name="${lr_prefix}_${fr_prefix}_shock">
+        <hardwareInterface>hardware_interface/EffortJointInterface</hardwareInterface>
+      </joint>
+      <actuator name="${lr_prefix}_${fr_prefix}_shock_act">
+        <mechanicalReduction>1</mechanicalReduction>
+      </actuator>
+    </transmission>
+  </xacro:macro>
+  <!-- The "wheel" macro defines an axle carrier, axle, and wheel. -->
+  <xacro:macro name="wheel" params="lr_prefix fr_prefix lr_reflect">
+    <link name="${lr_prefix}_${fr_prefix}_axle_carrier">
+	  <!-- visual>
+        <origin xyz="0 0 0"/>
+        <geometry>
+          <cylinder radius="0.1" length="0.1"/>
+        </geometry>
+	  </visual>
+	  <collision>
+        <origin xyz="0 0 0"/>
+        <geometry>
+          <cylinder radius="0.1" length="0.1"/>
+        </geometry>
+	  </collision -->
+      <xacro:null_inertial/>
+    </link>
+    <!-- The left and right axles have the same axis so that identical
+         rotation values cause the wheels to rotate in the same direction. -->
+    <joint name="${lr_prefix}_${fr_prefix}_axle" type="continuous">
+      <parent link="${lr_prefix}_${fr_prefix}_axle_carrier"/>
+      <child link="${lr_prefix}_${fr_prefix}_wheel"/>
+      <origin rpy="${degrees_90} 0 ${degrees_180}"/>
+      <axis xyz="0 0 -1"/>
+      <limit effort="${axle_eff_limit}" velocity="${axle_vel_limit}"/>
+      <joint_properties damping="${wheel_joint_damping}" friction="{wheel_joint_friction}"/>
+    </joint>
+    <transmission name="${lr_prefix}_${fr_prefix}_axle_trans">
+      <type>transmission_interface/SimpleTransmission</type>
+      <joint name="${lr_prefix}_${fr_prefix}_axle">
+        <!-- hardwareInterface>hardware_interface/EffortJointInterface</hardwareInterface -->
+        <hardwareInterface>hardware_interface/VelocityJointInterface</hardwareInterface>
+      </joint>
+      <actuator name="${lr_prefix}_${fr_prefix}_axle_act">
+        <mechanicalReduction>1</mechanicalReduction>
+      </actuator>
+    </transmission>
+    <gazebo reference="${lr_prefix}_${fr_prefix}_axle_carrier">
+      <material>Gazebo/Black</material>
+    </gazebo>
+    <link name="${lr_prefix}_${fr_prefix}_wheel">
+      <visual>
+        <origin xyz="0
+                     0
+                     ${lr_reflect * (axle_length - (tire_width / 2 - hex_hub_depth))}"/>
+        <geometry>
+          <cylinder radius="${tire_dia / 2}" length="${tire_width}"/>
+        </geometry>
+        <material name="tire_mat"/>
+      </visual>
+      <collision>
+        <origin xyz="0
+                     0
+                     ${lr_reflect * (axle_length - (tire_width / 2 - hex_hub_depth))}"/>
+        <geometry>
+          <cylinder radius="${tire_dia / 2}" length="${tire_width}"/>
+        </geometry>
+      </collision>
+      <xacro:thick_walled_tube_inertial
+          inner_rad="${hub_dia / 2}" outer_rad="${tire_dia / 2}"
+          height="${tire_width}" mass="${wheel_mass}"/>
+    </link>
+    <gazebo reference="${lr_prefix}_${fr_prefix}_wheel">
+      <material>Gazebo/Black</material>
+    </gazebo>
+  </xacro:macro>
+  <!-- xacro:macro name="rubber_wheel" params="name parent *origin reflect hq" -->
+  <!-- Front wheel -->
+  <xacro:macro name="front_wheel"
+               params="lr_prefix fr_prefix lr_reflect fr_reflect">
+    <xacro:shock_front lr_prefix="${lr_prefix}" fr_prefix="${fr_prefix}"
+                 lr_reflect="${lr_reflect}" fr_reflect="${fr_reflect}"
+                 child="${lr_prefix}_steering_link"/>
+    <link name="${lr_prefix}_steering_link">
+	  <!-- visual>
+		<origin xyz="0 0 0"/>
+        <geometry>
+          <cylinder radius="0.1" length="0.1"/>
+        </geometry>
+	  </visual>
+	  <collision>
+		<origin xyz="0 0 0"/>
+        <geometry>
+          <cylinder radius="0.1" length="0.1"/>
+        </geometry>
+	  </collision -->
+      <xacro:null_inertial/>
+    </link>
+    <joint name="${lr_prefix}_steering_joint" type="revolute">
+      <parent link="${lr_prefix}_steering_link"/>
+      <child link="${lr_prefix}_${fr_prefix}_axle_carrier"/>
+      <axis xyz="0 0 1"/>
+      <limit lower="${-degrees_45}" upper="${degrees_45}"
+             effort="${servo_stall_torque}" velocity="${servo_no_load_speed}"/>
+    </joint>
+    <transmission name="${lr_prefix}_steering_trans">
+      <type>transmission_interface/SimpleTransmission</type>
+      <joint name="${lr_prefix}_steering_joint">
+        <hardwareInterface>hardware_interface/EffortJointInterface</hardwareInterface>
+      </joint>
+      <actuator name="${lr_prefix}_steering_act">
+        <mechanicalReduction>1</mechanicalReduction>
+      </actuator>
+    </transmission>
+    <gazebo reference="${lr_prefix}_steering_link">
+      <material>Gazebo/Black</material>
+    </gazebo>
+    <xacro:wheel lr_prefix="${lr_prefix}" fr_prefix="${fr_prefix}"
+                 lr_reflect="${lr_reflect}"/>
+  </xacro:macro>
+  <!-- Rear wheel -->
+  <xacro:macro name="rear_wheel"
+               params="lr_prefix fr_prefix lr_reflect fr_reflect">
+    <xacro:shock lr_prefix="${lr_prefix}" fr_prefix="${fr_prefix}"
+                 lr_reflect="${lr_reflect}" fr_reflect="${fr_reflect}"
+                 child="${lr_prefix}_${fr_prefix}_axle_carrier"/>
+    <xacro:wheel lr_prefix="${lr_prefix}" fr_prefix="${fr_prefix}"
+                 lr_reflect="${lr_reflect}"/>
+  </xacro:macro>
 </robot>

File: niagara_model/urdf/DasAutonomeAuto.urdf (robot description, URDF)
Before this commit: robot dasautonomeauto, 2 links, 1 joints
Links:
- link base_link: geometry collision mesh filename=file://$(find niagara_model)/meshes/base_link_w_roof.STL; visual mesh filename=file://$(find niagara_model)/meshes/base_link_w_roof.STL

Commit message: niagara is launching correclty

File: niagara_model/urdf/Autoreifen.xacro (robot description, xacro)
@@ -6,7 +6,7 @@
        is a "zero offset" wheel. hex_hub_depth = tire_width / 2 -
        axle_length. -->
-    <xacro:property name="tire_dia" value="0.350"/>  <!-- Reduced from 0.440 -->
-    <xacro:property name="tire_width" value="0.195"/>  <!-- Reduced from 0.195 -->
-    <xacro:property name="hub_dia" value="0.235"/>  <!-- Reduced from 0.235 -->
+  <xacro:property name="tire_dia" value="0.350"/>  <!-- Reduced from 0.440 -->
+  <xacro:property name="tire_width" value="0.195"/>  <!-- Reduced from 0.195 -->
+  <xacro:property name="hub_dia" value="0.235"/>  <!-- Reduced from 0.235 -->
   <xacro:property name="hex_hub_depth" value="0.120"/> <!-- or +0.072 -->
   <xacro:property name="wheel_mass" value="8.0"/>   <!-- check -->
@@ -100,5 +100,5 @@
       <parent link="base_link"/>
       <child link="${child}"/>
-      <origin xyz="${fr_reflect * 0.90902595238888}
+      <origin xyz="${fr_reflect * 0.80902595238888}
                    ${lr_reflect * ((hex_hub_dist / 2) - axle_length)}
                    ${-wheel_travel}"/>

Commit message: the car go foward

File: niagara_model/urdf/Autoreifen.xacro (robot description, xacro)
@@ -142,5 +142,5 @@
       <child link="${lr_prefix}_${fr_prefix}_wheel"/>
       <origin rpy="${degrees_90} 0 ${degrees_180}"/>
-      <axis xyz="0 0 -1"/>
+      <axis xyz="0 0 1"/>
       <limit effort="${axle_eff_limit}" velocity="${axle_vel_limit}"/>
       <joint_properties damping="${wheel_joint_damping}" friction="{wheel_joint_friction}"/>

File: niagara_model/urdf/DasAutonomeAuto.urdf (robot description, URDF)
Before this commit: robot dasautonomeauto, 2 links, 1 joints
Links:
- link base_link: geometry collision mesh filename=file://$(find niagara_model)/meshes/base_link.STL; visual mesh filename=file://$(find niagara_model)/meshes/base_link.STL

File: niagara_model/urdf/sensors.xacro (robot description, xacro)
@@ -10,7 +10,5 @@
                 <param name="max">5</param>
             </command_interface>
-            <state_interface name="velocity"/>
             <state_interface name="position"/>
-            <state_interface name="effort"/>
         </joint>
         <joint name="left_steering_joint">
@@ -19,7 +17,37 @@
                 <param name="max">5</param>
             </command_interface>
+            <state_interface name="position"/>
+        </joint>
+        <joint name="left_rear_shock">
+            <command_interface name="effort">
+                <param name="min">-1</param>
+                <param name="max">1</param>
+            </command_interface>
+            <state_interface name="effort"/>
+        </joint>
+        <joint name="right_rear_shock">
+            <command_interface name="effort">
+                <param name="min">-1</param>
+                <param name="max">1</param>
+            </command_interface>
+            <state_interface name="effort"/>
+        </joint>
+        <joint name="left_front_shock">
+            <command_interface name="effort">
+                <param name="min">-1</param>
+                <param name="max">1</param>
+            </command_interface>
+            <state_interface name="effort"/>
+        </joint>
+        <joint name="right_front_shock">
+            <command_interface name="effort">
+                <param name="min">-1</param>
+                <param name="max">1</param>
+            </command_interface>
+            <state_interface name="effort"/>
+        </joint>
+        <joint name="left_rear_axle">
+            <command_interface name="velocity"/>
             <state_interface name="velocity"/>
-            <state_interface name="position"/>
-            <state_interface name="effort"/>
         </joint>
     </ros2_control>
