Commit message: urdf car uplouded

File: niagara_model/urdf/Autoreifen.xacro (robot description, xacro)
@@ -15,4 +15,13 @@
   <xacro:property name="front_wheel_y" value="0.495625727164768"/>
   <xacro:property name="front_wheel_z" value="0.1094929592556163"/>
+  <xacro:property name="rear_wheel_x" value="1.04780116842239"/>
+  <xacro:property name="rear_wheel_y" value="0.495625727164768"/>
+  <xacro:property name="rear_wheel_z" value="0.1094929592556163"/>
+  <!-- Degree-to-radian conversions -->
+  <xacro:property name="degrees_45" value="0.785398163"/>
+  <xacro:property name="degrees_90" value="1.57079633"/>
+  <xacro:property name="degrees_180" value="3.14159265"/>
+  <xacro:property name="servo_stall_torque" value="50"/>  <!-- check -->
+  <xacro:property name="servo_no_load_speed" value="25"/> <!-- check -->
   <xacro:macro name="thick_walled_tube_inertial"
                params="inner_rad outer_rad height mass">
@@ -35,6 +44,49 @@
     </inertial>
   </xacro:macro>
-    <!-- front wheel -->
+  <!-- front wheel -->
   <xacro:macro name="front_wheel" params="lr_prefix fr_prefix lr_reflect">
+    <link name="${lr_prefix}_steering_link">
+      <xacro:null_inertial/>
+    </link>
+    <joint name="${lr_prefix}_steering_joint" type="revolute">
+      <origin xyz="${fr_reflect * front_wheel_x} ${lr_reflect * front_wheel_y} ${-front_wheel_z}" rpy="0 ${degrees_90} 0"/>
+      <parent link="base_link"/>
+      <child link="${lr_prefix}_steering_link"/>
+      <axis xyz="-1 0 0"/>
+      <limit lower="${-degrees_45}" upper="${degrees_45}"
+            effort="${servo_stall_torque}" velocity="${servo_no_load_speed}"/>
+    </joint>
+    <link name="${lr_prefix}_${fr_prefix}_wheel">
+      <visual>
+        <origin xyz="0
+                     0
+                     ${lr_reflect * ((tire_width / 2 - hex_hub_depth))}" rpy="0 0 0"/>
+        <geometry>
+          <cylinder radius="${tire_dia / 2}" length="${tire_width}"/>
+        </geometry>
+        <material name="tire_mat"/>
+      </visual>
+      <collision>
+        <origin xyz="0
+                     0
+                     ${lr_reflect * ((tire_width / 2 - hex_hub_depth))}" rpy="0 0 0"/>
+        <geometry>
+          <cylinder radius="${tire_dia / 2}" length="${tire_width}"/>
+        </geometry>
+      </collision>
+      <xacro:thick_walled_tube_inertial
+          inner_rad="${hub_dia / 2}" outer_rad="${tire_dia / 2}"
+          height="${tire_width}" mass="${wheel_mass}"/>
+    </link>
+    <joint name="${lr_prefix}_${fr_prefix}_axle" type="continuous">
+      <parent link="${lr_prefix}_steering_link"/>
+      <child link="${lr_prefix}_${fr_prefix}_wheel"/>
+      <origin xyz="0 0 0" rpy="1.5708 0 0" />
+      <axis xyz="0 0 -1"/>
+      <limit effort="${axle_eff_limit}" velocity="${axle_vel_limit}"/>
+    </joint>
+  </xacro:macro>
+  <!-- rear wheel -->
+  <xacro:macro name="rear_wheel" params="lr_prefix fr_prefix lr_reflect">
     <link name="${lr_prefix}_${fr_prefix}_wheel">
       <visual>
@@ -62,5 +114,5 @@
       <parent link="base_link"/>
       <child link="${lr_prefix}_${fr_prefix}_wheel"/>
-      <origin xyz="${fr_reflect * front_wheel_x} ${lr_reflect * front_wheel_y} ${-front_wheel_z}" rpy="1.5708 0 0"/>
+      <origin xyz="${fr_reflect * rear_wheel_x} ${lr_reflect * rear_wheel_y} ${-rear_wheel_z}" rpy="1.5708 0 0"/>
       <axis xyz="0 0 -1"/>
       <limit effort="${axle_eff_limit}" velocity="${axle_vel_limit}"/>
@@ -68,8 +120,8 @@
   </xacro:macro>
     <xacro:macro name="front_wheel_to_base" params="lr_prefix fr_prefix lr_reflect fr_reflect">
-        <xacro:front_wheel lr_prefix="${lr_prefix}" fr_prefix="${fr_prefix}" lr_reflect="${lr_reflect}"/>
+      <xacro:front_wheel lr_prefix="${lr_prefix}" fr_prefix="${fr_prefix}" lr_reflect="${lr_reflect}"/>
     </xacro:macro>
-    <!-- <xacro:macro name="rear_wheel" params="lr_prefix fr_prefix lr_reflect fr_reflect">
-        <xacro:wheel lr_prefix="${lr_prefix}" fr_prefix="${fr_prefix}" lr_reflect="${lr_reflect}"/>
-    </xacro:macro> -->
+    <xacro:macro name="rear_wheel_to_base" params="lr_prefix fr_prefix lr_reflect fr_reflect">
+        <xacro:rear_wheel lr_prefix="${lr_prefix}" fr_prefix="${fr_prefix}" lr_reflect="${lr_reflect}"/>
+    </xacro:macro>
 </robot>

File: niagara_model/urdf/Autoreifen_with_suspetion.xacro (robot description, xacro)
@@ -188,5 +188,5 @@
   <!-- Front wheel -->
   <xacro:macro name="front_wheel"
-               params="lr_prefix fr_prefix lr_reflect fr_reflect">
+               params="lrparams_prefix fr_prefix lr_reflect fr_reflect">
     <xacro:shock_front lr_prefix="${lr_prefix}" fr_prefix="${fr_prefix}"
                  lr_reflect="${lr_reflect}" fr_reflect="${fr_reflect}"
@@ -239,2 +239,83 @@
   </xacro:macro>
 </robot>
+<?xml version="1.0"?>
+<robot name="dasautonomeauto" xmlns:xacro="http://www.ros.org/wiki/xacro">
+  <xacro:property name="tire_dia" value="0.350"/>  <!-- Reduced from 0.440 -->
+  <xacro:property name="tire_width" value="0.195"/>  <!-- Reduced from 0.195 -->
+  <xacro:property name="hub_dia" value="0.235"/>  <!-- Reduced from 0.235 -->
+  <xacro:property name="hex_hub_depth" value="0.120"/> <!-- or +0.072 -->
+  <xacro:property name="wheel_mass" value="8.0"/>   <!-- check -->
+  <xacro:property name="wheelbase" value="2.1"/>
+  <xacro:property name="hex_hub_dist" value="0.9191"/>
+  <xacro:property name="wheel_travel" value="0.209492959255614"/>
+  <xacro:property name="axle_eff_limit" value="204.95"/>
+  <xacro:property name="axle_vel_limit" value="39.02"/>
+  <!-- Properties of the car -->
+  <xacro:property name="front_wheel_x" value="0.787346576344423"/>
+  <xacro:property name="front_wheel_y" value="0.495625727164768"/>
+  <xacro:property name="front_wheel_z" value="0.1094929592556163"/>
+  <!-- Degree-to-radian conversions -->
+  <xacro:property name="degrees_45" value="0.785398163"/>
+  <xacro:property name="degrees_90" value="1.57079633"/>
+  <xacro:property name="degrees_180" value="3.14159265"/>
+  <xacro:property name="servo_stall_torque" value="50"/>  <!-- check -->
+  <xacro:property name="servo_no_load_speed" value="25"/> <!-- check -->
+  <xacro:macro name="thick_walled_tube_inertial"
+               params="inner_rad outer_rad height mass">
+    <inertial>
+      <mass value="${mass}"/>
+      <inertia ixx="${(1 / 12) * mass * (3 * (inner_rad * inner_rad +
+                    outer_rad * outer_rad) + height * height)}"
+               ixy="0" ixz="0"
+               iyy="${(1 / 12) * mass * (3 * (inner_rad * inner_rad +
+                    outer_rad * outer_rad) + height * height)}"
+               iyz="0"
+               izz="${mass * (inner_rad * inner_rad +
+                    outer_rad * outer_rad) / 2}"/>
+    </inertial>
+  </xacro:macro>
+  <xacro:macro name="null_inertial">
+    <inertial>
+      <mass value="0.001"/>
+      <inertia ixx="0.001" ixy="0" ixz="0" iyy="0.001" iyz="0" izz="0.001"/>
+    </inertial>
+  </xacro:macro>
+    <!-- front wheel -->
+  <xacro:macro name="front_wheel" params="lr_prefix fr_prefix lr_reflect">
+    <link name="${lr_prefix}_${fr_prefix}_wheel">
+      <visual>
+        <origin xyz="0
+                     0
+                     ${lr_reflect * ((tire_width / 2 - hex_hub_depth))}" rpy="0 0 0"/>
+        <geometry>
+          <cylinder radius="${tire_dia / 2}" length="${tire_width}"/>
+        </geometry>
+        <material name="tire_mat"/>
+      </visual>
+      <collision>
+        <origin xyz="0
+                     0
+                     ${lr_reflect * ((tire_width / 2 - hex_hub_depth))}" rpy="0 0 0"/>
+        <geometry>
+          <cylinder radius="${tire_dia / 2}" length="${tire_width}"/>
+        </geometry>
+      </collision>
+      <xacro:thick_walled_tube_inertial
+          inner_rad="${hub_dia / 2}" outer_rad="${tire_dia / 2}"
+          height="${tire_width}" mass="${wheel_mass}"/>
+    </link>
+    <joint name="${lr_prefix}_${fr_prefix}_axle" type="continuous">
+      <parent link="base_link"/>
+      <child link="${lr_prefix}_${fr_prefix}_wheel"/>
+      <origin xyz="${fr_reflect * front_wheel_x} ${lr_reflect * front_wheel_y} ${-front_wheel_z}" rpy="1.5708 0 0"/>
+      <axis xyz="0 0 -1"/>
+      <limit effort="${axle_eff_limit}" velocity="${axle_vel_limit}"/>
+    </joint>
+  </xacro:macro>
+    <xacro:macro name="front_wheel_to_base" params="lr_prefix fr_prefix lr_reflect fr_reflect">
+      <xacro:front_wheel lr_prefix="${lr_prefix}" fr_prefix="${fr_prefix}" lr_reflect="${lr_reflect}"/>
+    </xacro:macro>
+    <!-- <xacro:macro name="rear_wheel" params="lr_prefix fr_prefix lr_reflect fr_reflect">
+        <xacro:wheel lr_prefix="${lr_prefix}" fr_prefix="${fr_prefix}" lr_reflect="${lr_reflect}"/>
+    </xacro:macro> -->
+</robot>

Commit message: Controller and model changes
In the model I add an innertial value to this part: {lr_prefix}_steering_link. This help to do not move when steering

File: niagara_model/urdf/Autoreifen.xacro (robot description, xacro)
@@ -47,5 +47,8 @@
   <xacro:macro name="front_wheel" params="lr_prefix fr_prefix lr_reflect">
     <link name="${lr_prefix}_steering_link">
-      <xacro:null_inertial/>
+      <!-- <xacro:null_inertial/> -->
+      <xacro:thick_walled_tube_inertial
+          inner_rad="${hub_dia / 2}" outer_rad="${tire_dia / 2}"
+          height="${tire_width}" mass="${wheel_mass}"/>
     </link>
     <joint name="${lr_prefix}_steering_joint" type="revolute">

File: niagara_model/urdf/sensors.xacro (robot description, xacro)
@@ -21,4 +21,12 @@
             <state_interface name="position"/>
         </joint>
+        <joint name="left_front_axle">
+            <command_interface name="velocity"/>
+            <state_interface name="velocity"/>
+        </joint>
+        <joint name="right_front_axle">
+            <command_interface name="velocity"/>
+            <state_interface name="velocity"/>
+        </joint>
     </ros2_control>
     <gazebo>

Commit message: ackermann plug in added because the odometry was bad

File: niagara_model/urdf/Autoreifen.xacro (robot description, xacro)
@@ -24,4 +24,7 @@
   <xacro:property name="servo_stall_torque" value="50"/>  <!-- check -->
   <xacro:property name="servo_no_load_speed" value="25"/> <!-- check -->
+  <material name="black">
+      <color rgba="0 0 0 1"/>
+  </material>
   <xacro:macro name="thick_walled_tube_inertial"
                params="inner_rad outer_rad height mass">
@@ -40,5 +43,5 @@
   <xacro:macro name="null_inertial">
     <inertial>
-      <mass value="0.001"/>
+      <mass value="4.5"/>
       <inertia ixx="0.001" ixy="0" ixz="0" iyy="0.001" iyz="0" izz="0.001"/>
     </inertial>
@@ -47,8 +50,8 @@
   <xacro:macro name="front_wheel" params="lr_prefix fr_prefix lr_reflect">
     <link name="${lr_prefix}_steering_link">
-      <!-- <xacro:null_inertial/> -->
-      <xacro:thick_walled_tube_inertial
+      <xacro:null_inertial/>
+      <!-- <xacro:thick_walled_tube_inertial
           inner_rad="${hub_dia / 2}" outer_rad="${tire_dia / 2}"
-          height="${tire_width}" mass="${wheel_mass}"/>
+          height="${tire_width}" mass="${wheel_mass}"/> -->
     </link>
     <joint name="${lr_prefix}_steering_joint" type="revolute">
@@ -68,5 +71,5 @@
           <cylinder radius="${tire_dia / 2}" length="${tire_width}"/>
         </geometry>
-        <material name="tire_mat"/>
+        <material name="black" />
       </visual>
       <collision>
@@ -100,5 +103,5 @@
           <cylinder radius="${tire_dia / 2}" length="${tire_width}"/>
         </geometry>
-        <material name="tire_mat"/>
+        <material name="black" />
       </visual>
       <collision>

Commit message: zed camara added

File: niagara_model/urdf/Autoreifen.xacro (robot description, xacro)
@@ -92,4 +92,7 @@
       <limit effort="${axle_eff_limit}" velocity="${axle_vel_limit}"/>
     </joint>
+    <gazebo reference="${lr_prefix}_${fr_prefix}_wheel">
+      <material>Gazebo/Black</material>
+    </gazebo>
   </xacro:macro>
   <!-- rear wheel -->
@@ -124,4 +127,7 @@
       <limit effort="${axle_eff_limit}" velocity="${axle_vel_limit}"/>
     </joint>
+    <gazebo reference="${lr_prefix}_${fr_prefix}_wheel">
+      <material>Gazebo/Black</material>
+    </gazebo>
   </xacro:macro>
     <xacro:macro name="front_wheel_to_base" params="lr_prefix fr_prefix lr_reflect fr_reflect">

File: niagara_model/urdf/VLP-16.xacro (robot description, xacro)
@@ -54,4 +54,5 @@
     <!-- Gazebo requires the velodyne_gazebo_plugins package -->
     <gazebo reference="${name}">
+    <material>Gazebo/Red</material>
       <xacro:if value="${gpu}">
         <sensor type="gpu_ray" name="${name}-VLP16">
