Commit message: sds

File: niagara_model/urdf/zed2.xacro (robot description, xacro)
@@ -8,5 +8,5 @@
         <parent link="base_link"/>
         <child link="zed_camera_link"/>
-        <origin xyz="0.6 0 0.5" rpy="0 0 0"/>
+        <origin xyz="0.6 0 0.6" rpy="0 0 0"/>
     </joint>
     <link name="zed_camera_link">
